Commit message: Add camera.xacro for camera integration and update materials in bot.xacro

File: bot_description/urdf/bot.xacro (robot description, xacro)
@@ -4,4 +4,5 @@
 <xacro:include filename="$(find bot_description)/urdf/bot.trans" />
 <xacro:include filename="$(find bot_description)/urdf/bot.gazebo" />
+<xacro:include filename="$(find bot_description)/urdf/camera.xacro" />
 <link name="base_footprint">
   <!-- <collision>
@@ -49,5 +50,5 @@
       <mesh filename="file://$(find bot_description)/meshes/right_wheel_1.stl" scale="0.001 0.001 0.001"/>
     </geometry>
-    <material name="silver"/>
+    <material name="black"/>
   </visual>
   <collision>
@@ -89,5 +90,5 @@
       <mesh filename="file://$(find bot_description)/meshes/left_wheel_1.stl" scale="0.001 0.001 0.001"/>
     </geometry>
-    <material name="silver"/>
+    <material name="black"/>
   </visual>
   <collision>

File: bot_description/urdf/materials.xacro (robot description, xacro)
@@ -4,3 +4,9 @@
   <color rgba="0.700 0.700 0.700 1.000"/>
 </material>
+<material name="black">
+    <color rgba="0 0 0 1"/>
+</material>
+<material name="Green">
+    <color rgba="0 1 0 1"/>
+</material>
 </robot>

Commit message: Update README and Xacro files: add depth camera support and correct materials

File: bot_description/urdf/bot.xacro (robot description, xacro)
@@ -4,5 +4,6 @@
 <xacro:include filename="$(find bot_description)/urdf/bot.trans" />
 <xacro:include filename="$(find bot_description)/urdf/bot.gazebo" />
-<xacro:include filename="$(find bot_description)/urdf/camera.xacro" />
+<!-- <xacro:include filename="$(find bot_description)/urdf/camera.xacro" /> -->
+<xacro:include filename="$(find bot_description)/urdf/depth_camera.xacro" />
 <link name="base_footprint">
   <!-- <collision>

File: bot_description/urdf/materials.xacro (robot description, xacro)
@@ -1,12 +1,15 @@
 <?xml version="1.0" ?>
-<robot name="bot" xmlns:xacro="http://www.ros.org/wiki/xacro" >
-<material name="silver">
-  <color rgba="0.700 0.700 0.700 1.000"/>
-</material>
-<material name="black">
+<robot name="bot" xmlns:xacro="http://www.ros.org/wiki/xacro">
+  <material name="silver">
+    <color rgba="0.700 0.700 0.700 1.000"/>
+  </material>
+  <material name="black">
     <color rgba="0 0 0 1"/>
-</material>
-<material name="Green">
+  </material>
+  <material name="green">
     <color rgba="0 1 0 1"/>
-</material>
+  </material>
+  <material name="red">
+    <color rgba="1 0 0 1"/>
+  </material>
 </robot>
